Commit message: Update URDF with kinect.  Add Course World For Gazebo.

File: victor_description/robots/victor.urdf (robot description, URDF)
Before this commit: robot victor, 7 links, 6 joints
Links:
- added link base_kinect; visual box size=0.08 0.28 0.04
Joints:
- added joint kinect_joint: type fixed, parent base_link, child base_kinect, origin xyz=-0.105 0 0.5 rpy=0 0.52 0, axis 0 0 0
